Commit message: added gripper model

File: tests/urdfGen.urdf (robot description, URDF)
Before this commit: robot TEST, 11 links, 10 joints
Joints:
- joint fixed_0: child link_1 -> casing_0; parent casing_0 -> link_0
- joint fixed_1: child link_2 -> casing_1; origin xyz=0  0  0 rpy=0  0  0 -> xyz=0  0  1 rpy=1.5708           0      1.5708; parent casing_1 -> link_1
- joint fixed_2: child link_3 -> casing_2; origin xyz=0  0  0 rpy=0  0  0 -> xyz=0  0  0 rpy=-1.5708           0      1.5708; parent casing_2 -> link_2
- joint fixed_3: child link_4 -> casing_3; origin xyz=0  0  0 rpy=0  0  0 -> xyz=0.5           0           0 rpy=1.5708           0           0; parent casing_3 -> link_3
- joint fixed_4: child link_5 -> casing_4; origin xyz=0  0  0 rpy=0  0  0 -> xyz=0  0  0 rpy=-1.5708           0           0; parent casing_4 -> link_4
- joint joint_0: child casing_0 -> link_1; parent link_0 -> casing_0
- joint joint_1: child casing_1 -> link_2; origin xyz=0  0  1 rpy=1.5708           0      1.5708 -> xyz=0  0  0 rpy=0  0  0; parent link_1 -> casing_1
- joint joint_2: child casing_2 -> link_3; origin xyz=0  0  0 rpy=-1.5708           0      1.5708 -> xyz=0  0  0 rpy=0  0  0; parent link_2 -> casing_2
- joint joint_3: child casing_3 -> link_4; origin xyz=0.5           0           0 rpy=1.5708           0           0 -> xyz=0  0  0 rpy=0  0  0; parent link_3 -> casing_3
- joint joint_4: child casing_4 -> link_5; origin xyz=0  0  0 rpy=-1.5708           0           0 -> xyz=0  0  0 rpy=0  0  0; parent link_4 -> casing_4

File: tests/urdfGen_1.urdf (robot description, URDF)
Before this commit: robot TEST, 8 links, 7 joints
Links:
- added link gripper_case, mass 0; collision box size=0.025 0.025 0.05; visual box size=0.025 0.025 0.05
- added link jaw_1, mass 0.001; collision box size=0.0125 0.0125 0.05; visual box size=0.0125 0.0125 0.05
- added link jaw_2, mass 0.001; collision box size=0.0125 0.0125 0.05; visual box size=0.0125 0.0125 0.05
Joints:
- added joint fixed_ee_2: type fixed, parent link_3, child jaw_2, origin xyz=0.5           0           0 rpy=3.1416           0           0, axis 0  0  1, limit lower=0 upper=0 effort=1000000 velocity=1000000
- added joint gripper: type prismatic, parent gripper_case, child jaw_1, origin xyz=0  0  0 rpy=0  0  0, axis 0  0  1, limit lower=-0.1 upper=0 effort=1000000 velocity=1000000
- added joint gripper_fixed: type fixed, parent link_3, child gripper_case, origin xyz=0.5           0           0 rpy=3.1416           0           0, axis 0  0  1, limit lower=0 upper=0 effort=1000000 velocity=1000000
- joint fixed_0: child link_1 -> casing_0; parent casing_0 -> link_0
- joint fixed_1: child link_2 -> casing_1; origin xyz=0  0  0 rpy=0  0  0 -> xyz=0.5           0           0 rpy=1.5708           0           0; parent casing_1 -> link_1_L
- joint fixed_2: child link_3 -> casing_2; origin xyz=0  0  0 rpy=0  0  0 -> xyz=0.5           0           0 rpy=0  0  0; parent casing_2 -> link_2
- joint joint_0: child casing_0 -> link_1; parent link_0 -> casing_0
- joint joint_1: child casing_1 -> link_2; origin xyz=0.5           0           0 rpy=1.5708           0           0 -> xyz=0  0  0 rpy=0  0  0; parent link_1_L -> casing_1
- joint joint_2: child casing_2 -> link_3; origin xyz=0.5           0           0 rpy=0  0  0 -> xyz=0  0  0 rpy=0  0  0; parent link_2 -> casing_2

File: tests/urdfGen_10.urdf (robot description, URDF)
Before this commit: robot TEST, 21 links, 20 joints
Links:
- added link gripper_case, mass 0; collision box size=0.005 0.005 0.01; visual box size=0.005 0.005 0.01
- added link jaw_1, mass 0.001; collision box size=0.0025 0.0025 0.01; visual box size=0.0025 0.0025 0.01
- added link jaw_2, mass 0.001; collision box size=0.0025 0.0025 0.01; visual box size=0.0025 0.0025 0.01
Joints:
- added joint fixed_ee_2: type fixed, parent link_10, child jaw_2, origin xyz=0           0        0.05 rpy=-1.5708     -1.5708           0, axis 0  0  1, limit lower=0 upper=0 effort=1000000 velocity=1000000
- added joint gripper: type prismatic, parent gripper_case, child jaw_1, origin xyz=0  0  0 rpy=0  0  0, axis 0  0  1, limit lower=-0.02 upper=0 effort=1000000 velocity=1000000
- added joint gripper_fixed: type fixed, parent link_10, child gripper_case, origin xyz=0           0        0.05 rpy=-1.5708     -1.5708           0, axis 0  0  1, limit lower=0 upper=0 effort=1000000 velocity=1000000
- joint fixed_0: child link_1 -> casing_0; parent casing_0 -> link_0
- joint fixed_1: child link_2 -> casing_1; origin xyz=0  0  0 rpy=0  0  0 -> xyz=0           0        0.15 rpy=1.5708           0           0; parent casing_1 -> link_1
- joint fixed_2: child link_3 -> casing_2; origin xyz=0  0  0 rpy=0  0  0 -> xyz=3.0616e-18        0.05           0 rpy=1.5708           0      1.5708; parent casing_2 -> link_2
- joint fixed_3: child link_4 -> casing_3; origin xyz=0  0  0 rpy=0  0  0 -> xyz=0.05           0           0 rpy=-1.5708           0           0; parent casing_3 -> link_3
- joint fixed_4: child link_5 -> casing_4; origin xyz=0  0  0 rpy=0  0  0 -> xyz=0.05           0           0 rpy=1.5708           0           0; parent casing_4 -> link_4
- joint fixed_5: child link_6 -> casing_5; origin xyz=0  0  0 rpy=0  0  0 -> xyz=0.05           0           0 rpy=-1.5708           0           0; parent casing_5 -> link_5
- joint fixed_6: child link_7 -> casing_6; origin xyz=0  0  0 rpy=0  0  0 -> xyz=0.05           0           0 rpy=1.5708           0           0; parent casing_6 -> link_6
- joint fixed_7: child link_8 -> casing_7; origin xyz=0  0  0 rpy=0  0  0 -> xyz=0.05           0           0 rpy=-1.5708           0           0; parent casing_7 -> link_7
- joint fixed_8: child link_9 -> casing_8; origin xyz=0  0  0 rpy=0  0  0 -> xyz=0.05           0           0 rpy=1.5708           0           0; parent casing_8 -> link_8
- joint fixed_9: child link_10 -> casing_9; origin xyz=0  0  0 rpy=0  0  0 -> xyz=0  0  0 rpy=1.5708           0      1.5708; parent casing_9 -> link_9
- joint joint_0: child casing_0 -> link_1; parent link_0 -> casing_0
- joint joint_1: child casing_1 -> link_2; origin xyz=0           0        0.15 rpy=1.5708           0           0 -> xyz=0  0  0 rpy=0  0  0; parent link_1 -> casing_1
- joint joint_2: child casing_2 -> link_3; origin xyz=3.0616e-18        0.05           0 rpy=1.5708           0      1.5708 -> xyz=0  0  0 rpy=0  0  0; parent link_2 -> casing_2
- joint joint_3: child casing_3 -> link_4; origin xyz=0.05           0           0 rpy=-1.5708           0           0 -> xyz=0  0  0 rpy=0  0  0; parent link_3 -> casing_3
- joint joint_4: child casing_4 -> link_5; origin xyz=0.05           0           0 rpy=1.5708           0           0 -> xyz=0  0  0 rpy=0  0  0; parent link_4 -> casing_4
- joint joint_5: child casing_5 -> link_6; origin xyz=0.05           0           0 rpy=-1.5708           0           0 -> xyz=0  0  0 rpy=0  0  0; parent link_5 -> casing_5
- joint joint_6: child casing_6 -> link_7; origin xyz=0.05           0           0 rpy=1.5708           0           0 -> xyz=0  0  0 rpy=0  0  0; parent link_6 -> casing_6
- joint joint_7: child casing_7 -> link_8; origin xyz=0.05           0           0 rpy=-1.5708           0           0 -> xyz=0  0  0 rpy=0  0  0; parent link_7 -> casing_7
- joint joint_8: child casing_8 -> link_9; origin xyz=0.05           0           0 rpy=1.5708           0           0 -> xyz=0  0  0 rpy=0  0  0; parent link_8 -> casing_8
- joint joint_9: child casing_9 -> link_10; origin xyz=0  0  0 rpy=1.5708           0      1.5708 -> xyz=0  0  0 rpy=0  0  0; parent link_9 -> casing_9
